Commit message: gz_mv_launcher load_yaml() corregido y world

File: src/hexapod_description/urdf/hexapod_gz_properties.xacro (robot description, xacro)
@@ -1,6 +1,5 @@
 <robot name="hexapod" xmlns:xacro="http://ros.org/wiki/xacro">
   <gazebo reference="base_link">
-  <!-- =====================
-    <material>Gazebo/White</material>-->
+    <material>Gazebo/White</material>
     <mu1 value="1.0" />
     <mu2 value="1.0" />

File: src/hexapod_description/urdf/hexapod_urdf.ros2_control.xacro (robot description, xacro)
@@ -4,4 +4,5 @@
     <hardware>
       <!-- Hardware falso para simulación -->
+      <plugin>mock_components/GenericSystem</plugin>
       <plugin>gazebo_ros2_control/GazeboSystem</plugin>
     </hardware>

File: src/hexapod_description/urdf/hexapod_urdf.xacro (robot description, xacro)
@@ -103,5 +103,5 @@
       <child link="${prefix}_linkA"/>
       <axis xyz="${axisAx} ${axisAy} ${axisAz}"/>
-      <limit  lower="${lowerA}" upper="${upperA}" effort="10" velocity="1.0"/>
+      <limit effort="20.0" lower="${lowerA}" upper="${upperA}" velocity="1.0"/>
       <dynamics damping="0.5" friction="0.1"/>
     </joint>
@@ -133,5 +133,5 @@
       <child link="${prefix}_linkB"/>
       <axis xyz="${axisBx} ${axisBy} ${axisBz}"/>
-      <limit  lower="${lowerB}" upper="${upperB}" effort="10" velocity="1.0"/>
+      <limit effort="20.0" lower="${lowerB}" upper="${upperB}" velocity="1.0"/>
       <dynamics damping="0.5" friction="0.1"/>
     </joint>
@@ -163,5 +163,5 @@
       <child link="${prefix}_linkC"/>
       <axis xyz="${axisCx} ${axisCy} ${axisCz}"/>
-      <limit  lower="${lowerC}" upper="${upperC}" effort="10" velocity="1.0"/>
+      <limit effort="20.0" lower="${lowerC}" upper="${upperC}" velocity="1.0"/>
       <dynamics damping="0.5" friction="0.1"/>
     </joint>
@@ -369,3 +369,4 @@
                            stlP_path="package://hexapod_description/meshes/6P_link.STL"
   />
+  <xacro:include filename="$(find hexapod_description)/urdf/hexapod_urdf.ros2_control.xacro"/>
 </robot>

File: src/hexapod_moveit_config_new/config/hexapod.ros2_control.xacro (robot description, xacro)
@@ -6,5 +6,5 @@
             <hardware>
                 <!-- By default, set up controllers for simulation. This won't work on real hardware -->
-                <plugin>gazebo_ros2_control/GazeboSystem</plugin>
+                <plugin>mock_components/GenericSystem</plugin>
             </hardware>
             <joint name="leg1_jointA">

File: src/hexapod_moveit_config_new/config/hexapod.urdf.xacro (robot description, xacro)
@@ -1,84 +1,9 @@
 <?xml version="1.0"?>
 <robot xmlns:xacro="http://www.ros.org/wiki/xacro" name="hexapod">
-  <!-- ========================= -->
-  <!-- Arguments -->
-  <!-- ========================= -->
-  <!-- Switch: false = MoveIt/RViz, true = Gazebo -->
-  <xacro:arg name="use_gazebo" default="false"/>
-  <xacro:arg
-    name="initial_positions_file"
-    default="$(find hexapod_moveit_config_new)/config/initial_positions.yaml"/>
-  <!-- ========================= -->
-  <!-- Robot model -->
-  <!-- ========================= -->
-  <!-- Main hexapod geometry + joints -->
-  <xacro:include filename="$(find hexapod_description)/urdf/hexapod_urdf.xacro"/>
-  <!-- ros2_control definition -->
-  <xacro:include filename="$(find hexapod_moveit_config_new)/config/hexapod.ros2_control.xacro"/>
-  <!-- ========================= -->
-  <!-- TRANSMISSIONS (🔥 LO QUE FALTABA 🔥) -->
-  <!-- ========================= -->
-  <!-- Macro: effort transmission for Gazebo -->
-  <xacro:macro name="effort_transmission" params="joint_name">
-    <transmission name="${joint_name}_trans">
-      <type>transmission_interface/SimpleTransmission</type>
-      <joint name="${joint_name}">
-        <hardwareInterface>hardware_interface/EffortJointInterface</hardwareInterface>
-      </joint>
-      <actuator name="${joint_name}_motor">
-        <hardwareInterface>hardware_interface/EffortJointInterface</hardwareInterface>
-        <mechanicalReduction>1</mechanicalReduction>
-      </actuator>
-    </transmission>
-  </xacro:macro>
-  <!-- ========================= -->
-  <!-- Apply transmissions ONLY in Gazebo -->
-  <!-- ========================= -->
-  <xacro:if value="$(arg use_gazebo)">
-    <!-- Leg 1 -->
-    <xacro:effort_transmission joint_name="leg1_jointA"/>
-    <xacro:effort_transmission joint_name="leg1_jointB"/>
-    <xacro:effort_transmission joint_name="leg1_jointC"/>
-    <!-- Leg 2 -->
-    <xacro:effort_transmission joint_name="leg2_jointA"/>
-    <xacro:effort_transmission joint_name="leg2_jointB"/>
-    <xacro:effort_transmission joint_name="leg2_jointC"/>
-    <!-- Leg 3 -->
-    <xacro:effort_transmission joint_name="leg3_jointA"/>
-    <xacro:effort_transmission joint_name="leg3_jointB"/>
-    <xacro:effort_transmission joint_name="leg3_jointC"/>
-    <!-- Leg 4 -->
-    <xacro:effort_transmission joint_name="leg4_jointA"/>
-    <xacro:effort_transmission joint_name="leg4_jointB"/>
-    <xacro:effort_transmission joint_name="leg4_jointC"/>
-    <!-- Leg 5 -->
-    <xacro:effort_transmission joint_name="leg5_jointA"/>
-    <xacro:effort_transmission joint_name="leg5_jointB"/>
-    <xacro:effort_transmission joint_name="leg5_jointC"/>
-    <!-- Leg 6 -->
-    <xacro:effort_transmission joint_name="leg6_jointA"/>
-    <xacro:effort_transmission joint_name="leg6_jointB"/>
-    <xacro:effort_transmission joint_name="leg6_jointC"/>
-  </xacro:if>
-  <!-- ========================= -->
-  <!-- Control backends -->
-  <!-- ========================= -->
-  <!-- ===== MoveIt / RViz (NO Gazebo) ===== -->
-  <xacro:unless value="$(arg use_gazebo)">
-    <xacro:hexapod_ros2_control
-      name="FakeSystem"
-      initial_positions_file="$(arg initial_positions_file)"/>
-  </xacro:unless>
-  <gazebo>
-    <plugin name="gazebo_ros2_control" filename="libgazebo_ros2_control.so">
-      <robot_namespace>/</robot_namespace>
-      <parameters>$(find hexapod_moveit_config_new)/config/ros2_controllers.yaml</parameters>
-    </plugin>
-  </gazebo>
-  <!-- ===== Gazebo ===== -->
-  <xacro:if value="$(arg use_gazebo)">
-    <xacro:hexapod_ros2_control
-      name="HexapodSystem"
-      initial_positions_file="$(arg initial_positions_file)"/>
-  </xacro:if>
+    <xacro:arg name="initial_positions_file" default="initial_positions.yaml" />
+    <!-- Import hexapod urdf file -->
+    <xacro:include filename="$(find hexapod_description)/urdf/hexapod_urdf.xacro" />
+    <!-- Import control_xacro -->
+    <xacro:include filename="hexapod.ros2_control.xacro" />
+    <xacro:hexapod_ros2_control name="FakeSystem" initial_positions_file="$(arg initial_positions_file)"/>
 </robot>

Commit message: Corrección de doble inertia xx, vinculacion del urdf xacro con gz properties

File: src/hexapod_description/urdf/hexapod_gz_properties.xacro (robot description, xacro)
@@ -1,56 +1,27 @@
-<robot name="hexapod" xmlns:xacro="http://ros.org/wiki/xacro">
-  <gazebo reference="base_link">
-  <!-- =====================
-    <material>Gazebo/White</material>-->
-    <mu1 value="1.0" />
-    <mu2 value="1.0" />
+<?xml version="1.0"?>
+<robot xmlns:xacro="http://ros.org/wiki/xacro" name="hexapod">
+  <gazebo reference="leg1_linkP">
+    <mu1>1.8</mu1>
+    <mu2>1.8</mu2>
   </gazebo>
-  <gazebo reference="1C_link">
-    <mu1 value="1.0"/>
-    <mu2 value="1.0"/>
+  <gazebo reference="leg2_linkP">
+    <mu1>1.8</mu1>
+    <mu2>1.8</mu2>
   </gazebo>
-  <gazebo reference="2C_link">
-    <mu1 value="1.0"/>
-    <mu2 value="1.0"/>
+  <gazebo reference="leg3_linkP">
+    <mu1>1.8</mu1>
+    <mu2>1.8</mu2>
   </gazebo>
-  <gazebo reference="3C_link">
-    <mu1 value="1.0"/>
-    <mu2 value="1.0"/>
+  <gazebo reference="leg4_linkP">
+    <mu1>1.8</mu1>
+    <mu2>1.8</mu2>
   </gazebo>
-  <gazebo reference="4C_link">
-    <mu1 value="1.0"/>
-    <mu2 value="1.0"/>
+  <gazebo reference="leg5_linkP">
+    <mu1>1.8</mu1>
+    <mu2>1.8</mu2>
   </gazebo>
-  <gazebo reference="5C_link">
-    <mu1 value="1.0"/>
-    <mu2 value="1.0"/>
-  </gazebo>
-  <gazebo reference="6C_link">
-    <mu1 value="1.0"/>
-    <mu2 value="1.0"/>
-  </gazebo>
-  <gazebo reference="1P_link">
-    <mu1 value="1.0"/>
-    <mu2 value="1.0"/>
-  </gazebo>
-  <gazebo reference="2P_link">
-    <mu1 value="1.0"/>
-    <mu2 value="1.0"/>
-  </gazebo>
-  <gazebo reference="3P_link">
-    <mu1 value="1.0"/>
-    <mu2 value="1.0"/>
-  </gazebo>
-  <gazebo reference="4P_link">
-    <mu1 value="1.0"/>
-    <mu2 value="1.0"/>
-  </gazebo>
-  <gazebo reference="5P_link">
-    <mu1 value="1.0"/>
-    <mu2 value="1.0"/>
-  </gazebo>
-  <gazebo reference="6P_link">
-    <mu1 value="1.0"/>
-    <mu2 value="1.0"/>
+  <gazebo reference="leg6_linkP">
+    <mu1>1.8</mu1>
+    <mu2>1.8</mu2>
   </gazebo>
 </robot>

File: src/hexapod_description/urdf/hexapod_urdf.xacro (robot description, xacro)
@@ -103,6 +103,6 @@
       <child link="${prefix}_linkA"/>
       <axis xyz="${axisAx} ${axisAy} ${axisAz}"/>
-      <limit  lower="${lowerA}" upper="${upperA}" effort="10" velocity="1.0"/>
-      <dynamics damping="0.5" friction="0.1"/>
+      <limit  lower="${lowerA}" upper="${upperA}" effort="1.0" velocity="1.0"/>
+      <dynamics damping="1.0" friction="0.2"/>
     </joint>
     <link name="${prefix}_linkB">
@@ -133,6 +133,6 @@
       <child link="${prefix}_linkB"/>
       <axis xyz="${axisBx} ${axisBy} ${axisBz}"/>
-      <limit  lower="${lowerB}" upper="${upperB}" effort="10" velocity="1.0"/>
-      <dynamics damping="0.5" friction="0.1"/>
+      <limit  lower="${lowerB}" upper="${upperB}" effort="1.0" velocity="1.0"/>
+      <dynamics damping="1.0" friction="0.2"/>
     </joint>
     <link name="${prefix}_linkC">
@@ -163,12 +163,12 @@
       <child link="${prefix}_linkC"/>
       <axis xyz="${axisCx} ${axisCy} ${axisCz}"/>
-      <limit  lower="${lowerC}" upper="${upperC}" effort="10" velocity="1.0"/>
-      <dynamics damping="0.5" friction="0.1"/>
+      <limit  lower="${lowerC}" upper="${upperC}" effort="1.0" velocity="1.0"/>
+      <dynamics damping="1.0" friction="0.2"/>
     </joint>
     <link name="${prefix}_linkP">
       <inertial>
-        <mass value="0.001"/>
+        <mass value="0.002"/>
         <origin xyz="${origin_xP} ${origin_yP} ${origin_zP}" rpy="0 0 0"/>
-        <inertia ixx="${ixx_P}" ixy="${ixx_P}" ixz="${ixz_P}"
+        <inertia ixx="${ixx_P}" ixy="${ixy_P}" ixz="${ixz_P}"
                  iyy="${iyy_P}" iyz="${iyz_P}"
                  izz="${izz_P}"/>
@@ -369,3 +369,4 @@
                            stlP_path="package://hexapod_description/meshes/6P_link.STL"
   />
+  <xacro:include filename="$(find hexapod_description)/urdf/hexapod_gz_properties.xacro"/>
 </robot>
