Commit message: COmparacion con otro ws de hexapodo online, falta revisar launchers y urdfs, todo lo de moveit ya esta igual

File: src/hexapod_description/urdf/hexapod_urdf.xacro (robot description, xacro)
@@ -1,4 +1,9 @@
 <?xml version="1.0"?>
 <robot xmlns:xacro="http://ros.org/wiki/xacro" name="hexapod">
+  <!-- Hardware interface selection -->
+  <xacro:arg name="use_gazebo" default="false" />
+  <xacro:arg name="use_fake_hardware" default="false" />
+  <xacro:arg name="fake_sensor_commands" default="false" />
+ <!-- Properties -->
   <xacro:property name="mass_A" value="0.0329624385476769"/>
   <xacro:property name="mass_B" value="0.0491658081930703"/>
@@ -16,10 +21,5 @@
     <color rgba="0 1 0 1"/>
   </material>
-  <link name="base_footprint"/>
-  <joint name="base_footprint_joint" type="fixed">
-    <parent link="base_footprint"/>
-    <child link="base_link"/>
-    <origin xyz="0 0 0" rpy="0 0 0"/>
-  </joint>
+ <!-- Robot Construction -->
   <link name="base_link">
     <inertial>
@@ -369,3 +369,5 @@
                            stlP_path="package://hexapod_description/meshes/6P_link.STL"
   />
+  <xacro:include filename="package://hexapod_description/xacro/hexapod.gazebo.xacro"/>
+  <xacro:hexapod_gazebo prefix=""/>
 </robot>

File: src/hexapod_moveit_config_new/config/hexapod.urdf.xacro (robot description, xacro)
@@ -1,84 +1,20 @@
 <?xml version="1.0"?>
 <robot xmlns:xacro="http://www.ros.org/wiki/xacro" name="hexapod">
-  <!-- ========================= -->
-  <!-- Arguments -->
-  <!-- ========================= -->
-  <!-- Switch: false = MoveIt/RViz, true = Gazebo -->
-  <xacro:arg name="use_gazebo" default="false"/>
-  <xacro:arg
-    name="initial_positions_file"
-    default="$(find hexapod_moveit_config_new)/config/initial_positions.yaml"/>
-  <!-- ========================= -->
-  <!-- Robot model -->
-  <!-- ========================= -->
-  <!-- Main hexapod geometry + joints -->
-  <xacro:include filename="$(find hexapod_description)/urdf/hexapod_urdf.xacro"/>
-  <!-- ros2_control definition -->
-  <xacro:include filename="$(find hexapod_moveit_config_new)/config/hexapod.ros2_control.xacro"/>
-  <!-- ========================= -->
-  <!-- TRANSMISSIONS (🔥 LO QUE FALTABA 🔥) -->
-  <!-- ========================= -->
-  <!-- Macro: effort transmission for Gazebo -->
-  <xacro:macro name="effort_transmission" params="joint_name">
-    <transmission name="${joint_name}_trans">
-      <type>transmission_interface/SimpleTransmission</type>
-      <joint name="${joint_name}">
-        <hardwareInterface>hardware_interface/EffortJointInterface</hardwareInterface>
-      </joint>
-      <actuator name="${joint_name}_motor">
-        <hardwareInterface>hardware_interface/EffortJointInterface</hardwareInterface>
-        <mechanicalReduction>1</mechanicalReduction>
-      </actuator>
-    </transmission>
-  </xacro:macro>
-  <!-- ========================= -->
-  <!-- Apply transmissions ONLY in Gazebo -->
-  <!-- ========================= -->
-  <xacro:if value="$(arg use_gazebo)">
-    <!-- Leg 1 -->
-    <xacro:effort_transmission joint_name="leg1_jointA"/>
-    <xacro:effort_transmission joint_name="leg1_jointB"/>
-    <xacro:effort_transmission joint_name="leg1_jointC"/>
-    <!-- Leg 2 -->
-    <xacro:effort_transmission joint_name="leg2_jointA"/>
-    <xacro:effort_transmission joint_name="leg2_jointB"/>
-    <xacro:effort_transmission joint_name="leg2_jointC"/>
-    <!-- Leg 3 -->
-    <xacro:effort_transmission joint_name="leg3_jointA"/>
-    <xacro:effort_transmission joint_name="leg3_jointB"/>
-    <xacro:effort_transmission joint_name="leg3_jointC"/>
-    <!-- Leg 4 -->
-    <xacro:effort_transmission joint_name="leg4_jointA"/>
-    <xacro:effort_transmission joint_name="leg4_jointB"/>
-    <xacro:effort_transmission joint_name="leg4_jointC"/>
-    <!-- Leg 5 -->
-    <xacro:effort_transmission joint_name="leg5_jointA"/>
-    <xacro:effort_transmission joint_name="leg5_jointB"/>
-    <xacro:effort_transmission joint_name="leg5_jointC"/>
-    <!-- Leg 6 -->
-    <xacro:effort_transmission joint_name="leg6_jointA"/>
-    <xacro:effort_transmission joint_name="leg6_jointB"/>
-    <xacro:effort_transmission joint_name="leg6_jointC"/>
-  </xacro:if>
-  <!-- ========================= -->
-  <!-- Control backends -->
-  <!-- ========================= -->
-  <!-- ===== MoveIt / RViz (NO Gazebo) ===== -->
-  <xacro:unless value="$(arg use_gazebo)">
-    <xacro:hexapod_ros2_control
-      name="FakeSystem"
-      initial_positions_file="$(arg initial_positions_file)"/>
-  </xacro:unless>
-  <gazebo>
-    <plugin name="gazebo_ros2_control" filename="libgazebo_ros2_control.so">
-      <robot_namespace>/</robot_namespace>
-      <parameters>$(find hexapod_moveit_config_new)/config/ros2_controllers.yaml</parameters>
-    </plugin>
-  </gazebo>
-  <!-- ===== Gazebo ===== -->
-  <xacro:if value="$(arg use_gazebo)">
-    <xacro:hexapod_ros2_control
-      name="HexapodSystem"
-      initial_positions_file="$(arg initial_positions_file)"/>
-  </xacro:if>
+  <!-- MoveIt configuration for Gazebo simulation -->
+  <xacro:arg name="prefix" default="" />
+  <!-- Hardware interface selection for simulation -->
+   <xacro:arg name="use_gazebo" default="false" />
+   <xacro:arg name="use_fake_hardware" default="false" />
+   <xacro:arg name="fake_sensor_commands" default="false" />
+  <!-- Include main hexapod definition from description package -->
+  <xacro:include filename="$(find hexapod_description)/urdf/hexapod_urdf.xacro" />
+  <!-- Create complete hexapod robot for MoveIt simulation -->
+  <xacro:hexapod_urdf
+        use_sim="true"
+        prefix="$(arg prefix)"
+        use_gazebo="$(arg use_gazebo)"
+        use_fake_hardware="$(arg use_fake_hardware)"
+        fake_sensor_commands="$(arg fake_sensor_commands)"
+        port_name="$(arg port_name)"
+        baud_rate="$(arg baud_rate)" />
 </robot>

Commit message: Inicio webots

File: src/hexapod_description/urdf/hexapod_urdf.xacro (robot description, xacro)
@@ -47,5 +47,5 @@
       <geometry>
         <mesh
-          filename="package://hexapod_description/meshes/base_link.STL" />
+          filename="package://hexapod_description/meshes/base_link_collider.dae" />
       </geometry>
     </collision>
@@ -71,5 +71,6 @@
                                           axisAy axisBy axisCy  axisPy
                                           axisAz axisBz axisCz  axisPz
-                                          stlA_path stlB_path stlC_path   stlP_path
+                                          stlA_path stlB_path stlC_path  stlP_path
+                                          colA_path colB_path colC_path
                                           lowerA lowerB lowerC
                                           upperA upperB upperC
@@ -94,5 +95,5 @@
         <origin xyz="0 0 0" rpy="0 0 0"/>
         <geometry>
-          <mesh filename="${stlA_path}" />
+          <mesh filename="${colA_path}" />
         </geometry>
       </collision>
@@ -124,5 +125,5 @@
         <origin xyz="0 0 0" rpy="0 0 0"/>
         <geometry>
-          <mesh filename="${stlB_path}" />
+          <mesh filename="${colB_path}" />
         </geometry>
       </collision>
@@ -154,5 +155,5 @@
         <origin xyz="0 0 0" rpy="0 0 0"/>
         <geometry>
-          <mesh filename="${stlC_path}" />
+          <mesh filename="${colC_path}" />
         </geometry>
       </collision>
@@ -170,5 +171,5 @@
         <mass value="0.001"/>
         <origin xyz="${origin_xP} ${origin_yP} ${origin_zP}" rpy="0 0 0"/>
-        <inertia ixx="${ixx_P}" ixy="${ixx_P}" ixz="${ixz_P}"
+        <inertia ixx="${ixx_P}" ixy="${ixy_P}" ixz="${ixz_P}"
                  iyy="${iyy_P}" iyz="${iyz_P}"
                  izz="${izz_P}"/>
@@ -181,10 +182,4 @@
         <material name="${mat_name}"/>
       </visual>
-      <collision>
-        <origin xyz="0 0 0" rpy="0 0 0"/>
-        <geometry>
-          <mesh filename="${stlP_path}" />
-        </geometry>
-      </collision>
     </link>
     <joint name="${prefix}_jointP" type="fixed">
@@ -223,4 +218,7 @@
                            stlC_path="package://hexapod_description/meshes/1C_link.STL"
                            stlP_path="package://hexapod_description/meshes/1P_link.STL"
+                           colA_path="package://hexapod_description/meshes/1A_link_collider.dae"
+                           colB_path="package://hexapod_description/meshes/1B_link_collider.dae"
+                           colC_path="package://hexapod_description/meshes/1C_link_collider.dae"
   />
   <xacro:leg prefix="leg2"
@@ -251,5 +249,8 @@
                            stlB_path="package://hexapod_description/meshes/2B_link.STL"
                            stlC_path="package://hexapod_description/meshes/2C_link.STL"
-                           stlP_path="package://hexapod_description/meshes/2P_link.STL"
+                           stlP_path="package://hexapod_description/meshes/1P_link.STL"
+                           colA_path="package://hexapod_description/meshes/1A_link_collider.dae"
+                           colB_path="package://hexapod_description/meshes/1B_link_collider.dae"
+                           colC_path="package://hexapod_description/meshes/1C_link_collider.dae"
   />
   <xacro:leg prefix="leg3"
@@ -280,5 +281,8 @@
                            stlB_path="package://hexapod_description/meshes/3B_link.STL"
                            stlC_path="package://hexapod_description/meshes/3C_link.STL"
-                           stlP_path="package://hexapod_description/meshes/3P_link.STL"
+                           stlP_path="package://hexapod_description/meshes/1P_link.STL"
+                           colA_path="package://hexapod_description/meshes/1A_link_collider.dae"
+                           colB_path="package://hexapod_description/meshes/1B_link_collider.dae"
+                           colC_path="package://hexapod_description/meshes/1C_link_collider.dae"
   />
   <xacro:leg prefix="leg4"
@@ -309,5 +313,8 @@
                            stlB_path="package://hexapod_description/meshes/4B_link.STL"
                            stlC_path="package://hexapod_description/meshes/4C_link.STL"
-                           stlP_path="package://hexapod_description/meshes/4P_link.STL"
+                           stlP_path="package://hexapod_description/meshes/1P_link.STL"
+                           colA_path="package://hexapod_description/meshes/1A_link_collider.dae"
+                           colB_path="package://hexapod_description/meshes/1B_link_collider.dae"
+                           colC_path="package://hexapod_description/meshes/1C_link_collider.dae"
   />
   <xacro:leg prefix="leg5"
@@ -338,5 +345,8 @@
                            stlB_path="package://hexapod_description/meshes/5B_link.STL"
                            stlC_path="package://hexapod_description/meshes/5C_link.STL"
-                           stlP_path="package://hexapod_description/meshes/5P_link.STL"
+                           stlP_path="package://hexapod_description/meshes/1P_link.STL"
+                           colA_path="package://hexapod_description/meshes/1A_link_collider.dae"
+                           colB_path="package://hexapod_description/meshes/1B_link_collider.dae"
+                           colC_path="package://hexapod_description/meshes/1C_link_collider.dae"
   />
   <xacro:leg prefix="leg6"
@@ -367,5 +377,8 @@
                            stlB_path="package://hexapod_description/meshes/6B_link.STL"
                            stlC_path="package://hexapod_description/meshes/6C_link.STL"
-                           stlP_path="package://hexapod_description/meshes/6P_link.STL"
+                           stlP_path="package://hexapod_description/meshes/1P_link.STL"
+                           colA_path="package://hexapod_description/meshes/1A_link_collider.dae"
+                           colB_path="package://hexapod_description/meshes/1B_link_collider.dae"
+                           colC_path="package://hexapod_description/meshes/1C_link_collider.dae"
   />
 </robot>
